Commit message: xacro/urdfの修正

File: urdf/bumper/bumper_f120a.xacro (robot description, xacro)
@@ -20,10 +20,10 @@
   <xacro:property name="bumper_alu_frame_z_offset" value="0.0485" />
   <joint name="bumper_aluminum_frame_fixed_joint_1" type="fixed">
-    <origin xyz="${bumper_alu_frame_x_offset} ${bumper_alu_frame_y_offset} ${bumper_alu_frame_z_offset}" rpy="0 0 0" />
+    <origin xyz="${bumper_alu_frame_y_offset} ${-bumper_alu_frame_x_offset} ${bumper_alu_frame_z_offset}" rpy="0 0 -1.5708" />
     <parent link="base_link" />
     <child link="bumper_aluminum_frame_1" />
   </joint>
   <joint name="bumper_aluminum_frame_fixed_joint_2" type="fixed">
-    <origin xyz="${-bumper_alu_frame_x_offset} ${bumper_alu_frame_y_offset} ${bumper_alu_frame_z_offset}" rpy="0 0 0" />
+    <origin xyz="${bumper_alu_frame_y_offset} ${bumper_alu_frame_x_offset} ${bumper_alu_frame_z_offset}" rpy="0 0 -1.5708" />
     <parent link="base_link" />
     <child link="bumper_aluminum_frame_2" />

File: urdf/bumper/bumper_mega3.xacro (robot description, xacro)
@@ -19,10 +19,10 @@
   <xacro:property name="bumper_alu_frame_z_offset" value="0.03" />
   <joint name="bumper_aluminum_frame_fixed_joint_1" type="fixed">
-    <origin xyz="${bumper_alu_frame_x_offset} 0.0 ${bumper_alu_frame_z_offset}" rpy="0 0 0" />
+    <origin xyz="0.0 ${-bumper_alu_frame_x_offset} ${bumper_alu_frame_z_offset}" rpy="0 0 -1.5708" />
     <parent link="base_link" />
     <child link="bumper_aluminum_frame_1" />
   </joint>
   <joint name="bumper_aluminum_frame_fixed_joint_2" type="fixed">
-    <origin xyz="${-bumper_alu_frame_x_offset} 0.0 ${bumper_alu_frame_z_offset}" rpy="0 0 0" />
+    <origin xyz="0.0 ${bumper_alu_frame_x_offset} ${bumper_alu_frame_z_offset}" rpy="0 0 -1.5708" />
     <parent link="base_link" />
     <child link="bumper_aluminum_frame_2" />

File: urdf/cam_stay/cam_stay_f120a.xacro (robot description, xacro)
@@ -13,5 +13,5 @@
 -->
   <joint name="cam_stay_frame_joint" type="fixed">
-    <origin xyz="${0.0+cam_mount_frame_y_pos} ${0.157+cam_mount_frame_x_pos} ${0.1955+cam_mount_frame_z_pos}" rpy="0 0 1.5708" />
+    <origin xyz="${0.157+cam_mount_frame_x_pos} ${0.0+cam_mount_frame_y_pos} ${0.1955+cam_mount_frame_z_pos}" rpy="0 0 0" />
     <parent link="base_link" />
     <child link="cam_mount_frame" />

File: urdf/cam_stay/cam_stay_mega3.xacro (robot description, xacro)
@@ -6,5 +6,5 @@
   <xacro:property name="cam_mount_frame_z_pos" value="0.0" />
   <joint name="cam_stay_frame_joint" type="fixed">
-    <origin xyz="${0.0+cam_mount_frame_y_pos} ${0.143+cam_mount_frame_x_pos} ${0.155+cam_mount_frame_z_pos}" rpy="0 0 1.5708" />
+    <origin xyz="${0.143+cam_mount_frame_x_pos} ${-cam_mount_frame_y_pos} ${0.155+cam_mount_frame_z_pos}" rpy="0 0 0" />
     <parent link="base_link" />
     <child link="cam_mount_frame" />

File: urdf/lrf/tg30_f120a.xacro (robot description, xacro)
@@ -3,9 +3,9 @@
   <!-- placement of TG30 on Megarover F120A -->
   <!-- the mesh origin is at centerline of laser, x-axis facing forward -->
-  <xacro:property name="tg30_lrf_front_x_offset" value="0.0" />
-  <xacro:property name="tg30_lrf_front_y_offset" value="0.213" />
+  <xacro:property name="tg30_lrf_front_x_offset" value="0.213" />
+  <xacro:property name="tg30_lrf_front_y_offset" value="0.0" />
   <xacro:property name="tg30_lrf_front_z_offset" value="0.2214" />
-  <xacro:property name="tg30_lrf_back_x_offset" value="0.0" />
-  <xacro:property name="tg30_lrf_back_y_offset" value="-0.2680" />
+  <xacro:property name="tg30_lrf_back_x_offset" value="-0.2680" />
+  <xacro:property name="tg30_lrf_back_y_offset" value="0.0" />
   <xacro:property name="tg30_lrf_back_z_offset" value="0.2214" />
   <xacro:property name="tg30_center_of_mass_x" value="-0.004299" />
@@ -16,5 +16,5 @@
     <parent link="base_link" />
     <child link="front_lrf_link" />
-    <origin xyz="${tg30_lrf_front_x_offset} ${tg30_lrf_front_y_offset} ${tg30_lrf_front_z_offset}" rpy="0 0 ${pi/2}" />
+    <origin xyz="${tg30_lrf_front_x_offset} ${tg30_lrf_front_y_offset} ${tg30_lrf_front_z_offset}" rpy="0 0 0" />
   </joint>
   <link name="front_lrf_link">
@@ -44,5 +44,5 @@
     <parent link="base_link" />
     <child link="back_lrf_link" />
-    <origin xyz="${tg30_lrf_back_x_offset} ${tg30_lrf_back_y_offset} ${tg30_lrf_back_z_offset}" rpy="0 0 ${-pi/2}" />
+    <origin xyz="${tg30_lrf_back_x_offset} ${tg30_lrf_back_y_offset} ${tg30_lrf_back_z_offset}" rpy="0 0 ${pi}" />
   </joint>
   <link name="back_lrf_link">

File: urdf/lrf/tg30_mega3.xacro (robot description, xacro)
@@ -1,9 +1,9 @@
 <robot name="lrf_tg30_mega3" xmlns:xacro="http://ros.org/wiki/xacro">
   <xacro:include filename="$(find vs_rover_options_description)/urdf/lrf/tg30_mega3.gazebo" />
-  <xacro:property name="tg30_lrf_front_x_offset" value="0.0" />
-  <xacro:property name="tg30_lrf_front_y_offset" value="0.1990" />
+  <xacro:property name="tg30_lrf_front_x_offset" value="0.1990" />
+  <xacro:property name="tg30_lrf_front_y_offset" value="0.0" />
   <xacro:property name="tg30_lrf_front_z_offset" value="0.1809" />
-  <xacro:property name="tg30_lrf_back_x_offset" value="0.0" />
-  <xacro:property name="tg30_lrf_back_y_offset" value="-0.1690" />
+  <xacro:property name="tg30_lrf_back_x_offset" value="-0.1690" />
+  <xacro:property name="tg30_lrf_back_y_offset" value="0.0" />
   <xacro:property name="tg30_lrf_back_z_offset" value="0.1809" />
   <xacro:property name="tg30_center_of_mass_x" value="-0.004299" />
@@ -13,5 +13,5 @@
     <parent link="base_link" />
     <child link="front_lrf_link" />
-    <origin xyz="${tg30_lrf_front_x_offset} ${tg30_lrf_front_y_offset} ${tg30_lrf_front_z_offset}" rpy="0 0 ${pi/2}" />
+    <origin xyz="${tg30_lrf_front_x_offset} ${tg30_lrf_front_y_offset} ${tg30_lrf_front_z_offset}" rpy="0 0 0" />
   </joint>
   <link name="front_lrf_link">
@@ -40,5 +40,5 @@
     <parent link="base_link" />
     <child link="back_lrf_link" />
-    <origin xyz="${tg30_lrf_back_x_offset} ${tg30_lrf_back_y_offset} ${tg30_lrf_back_z_offset}" rpy="0 0 ${-pi/2}" />
+    <origin xyz="${tg30_lrf_back_x_offset} ${tg30_lrf_back_y_offset} ${tg30_lrf_back_z_offset}" rpy="0 0 ${-pi}" />
   </joint>
   <link name="back_lrf_link">

File: urdf/lrf/tg30_s40a_lb.xacro (robot description, xacro)
@@ -1,9 +1,9 @@
 <robot name="lrf_tg30_s40a_lb" xmlns:xacro="http://ros.org/wiki/xacro">
   <xacro:include filename="$(find vs_rover_options_description)/urdf/lrf/tg30_s40a_lb.gazebo" />
-  <xacro:property name="tg30_lrf_front_x_offset" value="0.0" />
-  <xacro:property name="tg30_lrf_front_y_offset" value="0.230" />
+  <xacro:property name="tg30_lrf_front_x_offset" value="0.230" />
+  <xacro:property name="tg30_lrf_front_y_offset" value="0.0" />
   <xacro:property name="tg30_lrf_front_z_offset" value="0.0879" />
-  <xacro:property name="tg30_lrf_back_x_offset" value="0.0" />
-  <xacro:property name="tg30_lrf_back_y_offset" value="-0.230" />
+  <xacro:property name="tg30_lrf_back_x_offset" value="-0.230" />
+  <xacro:property name="tg30_lrf_back_y_offset" value="0.0" />
   <xacro:property name="tg30_lrf_back_z_offset" value="0.0879" />
   <xacro:property name="tg30_center_of_mass_x" value="-0.004299" />
@@ -13,5 +13,5 @@
     <parent link="base_link" />
     <child link="front_lrf_link" />
-    <origin xyz="${tg30_lrf_front_x_offset} ${tg30_lrf_front_y_offset} ${tg30_lrf_front_z_offset}" rpy="0 0 ${pi/2}" />
+    <origin xyz="${tg30_lrf_front_x_offset} ${tg30_lrf_front_y_offset} ${tg30_lrf_front_z_offset}" rpy="0 0 0" />
   </joint>
   <link name="front_lrf_link">
@@ -40,5 +40,5 @@
     <parent link="base_link" />
     <child link="back_lrf_link" />
-    <origin xyz="${tg30_lrf_back_x_offset} ${tg30_lrf_back_y_offset} ${tg30_lrf_back_z_offset}" rpy="0 0 ${-pi/2}" />
+    <origin xyz="${tg30_lrf_back_x_offset} ${tg30_lrf_back_y_offset} ${tg30_lrf_back_z_offset}" rpy="0 0 ${pi}" />
   </joint>
   <link name="back_lrf_link">
