Commit message: Publish verified ROS 2 Jazzy and Gazebo Harmonic package
Import the qualified package files and use the public Jazzy clone URLs.

File: urdf/bumper/bumper_f120a.xacro (robot description, xacro)
@@ -29,86 +29,12 @@
     <child link="bumper_aluminum_frame_2" />
   </joint>
-  <xacro:macro name="bumper" params="prefix num xyz z_dir">
-    <joint name="bumper_${prefix}_${num}_joint" type="prismatic">
-      <parent link="bumper_baseboard_${prefix}_link" />
-      <child link="bumper_${prefix}_${num}_link" />
-      <origin xyz="${xyz}" rpy="0 0 ${radians(z_dir)}" />
-      <limit lower="0.0" upper="0.00157" effort="1" velocity="1.0" />
-      <axis xyz="0 1 0" />
-      <origin xyz="0 0 0" rpy="0 0 0" />
-      <dynamics damping="0.01" />
-    </joint>
-    <transmission name="bumper_${prefix}_${num}_trans">
-      <type>transmission_interface/SimpleTransmission</type>
-      <joint name="bumper_${prefix}_${num}_joint">
-        <hardwareInterface>hardware_interface/EffortJointInterface</hardwareInterface>
-      </joint>
-      <actuator name="bumper_${prefix}_${num}_motor">
-        <hardwareInterface>hardware_interface/EffortJointInterface</hardwareInterface>
-        <mechanismReduction>1</mechanismReduction>
-      </actuator>
-    </transmission>
-    <link name="bumper_${prefix}_${num}_link">
-      <inertial>
-        <origin xyz="0 0.005962 0" rpy="0 0 0" />
-        <mass value="0.025" />
-        <inertia ixx="0.000002386738" iyy="0.000036995" izz="0.000036094"
-          ixy="0.0" iyz="0.0"
-          ixz="0.0" />
-      </inertial>
-      <visual>
-        <origin xyz="0 0 0" rpy="0 0 ${-pi}" />
-        <geometry>
-          <mesh filename="package://vs_rover_options_description/meshes/bumper/f120a_bumper_link.stl" scale="0.001 0.001 0.001" />
-        </geometry>
-        <material name="silver" />
-      </visual>
-      <collision>
-        <origin xyz="0 0 0" rpy="0 0 ${-pi}" />
-        <geometry>
-          <mesh filename="package://vs_rover_options_description/meshes/bumper/f120a_bumper_link.stl" scale="0.001 0.001 0.001" />
-        </geometry>
-      </collision>
-    </link>
-    <gazebo reference="bumper_${prefix}_${num}_link">
-      <material>Gazebo/Silver</material>
-      <kp value="10000" />
-      <kd value="100" />
-    </gazebo>
-  </xacro:macro>
+  <!-- F120A mounting of the reusable, passive spring-loaded 120 mm bumper. -->
   <xacro:macro name="bumperbaseboard" params="prefix parent xyz z_dir">
-    <joint name="bumper_baseboard_${prefix}_joint" type="fixed">
-      <parent link="${parent}" />
-      <child link="bumper_baseboard_${prefix}_link" />
-      <origin xyz="${xyz}" rpy="0 0 ${radians(z_dir)}" />
-    </joint>
-    <link name="bumper_baseboard_${prefix}_link">
-      <inertial>
-        <origin xyz="0.001473 -0.003 -0.000343" rpy="0 0 0" />
-        <mass value="0.600" />
-        <inertia ixx="0.0001816" iyy="0.006071" izz="0.006228"
-          ixy="0.0" iyz="-0.000005910574"
-          ixz="0.0" />
-      </inertial>
-      <visual>
-        <origin xyz="0 0 0" rpy="0 0 ${-pi}" />
-        <geometry>
-          <mesh filename="package://vs_rover_options_description/meshes/bumper/f120a_bumper_plate.stl" scale="0.001 0.001 0.001" />
-        </geometry>
-        <material name="dark_silver" />
-      </visual>
-      <collision>
-        <origin xyz="0 0 0" rpy="0 0 ${-pi}" />
-        <geometry>
-          <mesh filename="package://vs_rover_options_description/meshes/bumper/f120a_bumper_plate.stl" scale="0.001 0.001 0.001" />
-        </geometry>
-      </collision>
-    </link>
-    <gazebo reference="bumper_baseboard_${prefix}_link">
-      <material>Gazebo/DarkGray</material>
-    </gazebo>
-    <xacro:bumper prefix="${prefix}" num="0" xyz="0.136 -0.024711 0.0025" z_dir="20" />
-    <xacro:bumper prefix="${prefix}" num="1" xyz="0 -0.0497 0.0025" z_dir="0" />
-    <xacro:bumper prefix="${prefix}" num="2" xyz="-0.136 -0.024711 0.0025" z_dir="-20" />
+    <xacro:property name="bumper120_prefix" value="${prefix}_" />
+    <xacro:property name="bumper120_parent" value="${parent}" />
+    <xacro:property name="bumper120_xyz" value="${xyz}" />
+    <!-- The former mesh used a -pi rotation; the common model faces local +Y. -->
+    <xacro:property name="bumper120_rpy" value="0 0 ${radians(z_dir) - pi}" />
+    <xacro:include filename="$(find vs_rover_options_description)/urdf/bumper/120bumper.xacro" />
   </xacro:macro>
 </robot>

File: urdf/bumper/bumper_mega3.xacro (robot description, xacro)
@@ -28,86 +28,15 @@
     <child link="bumper_aluminum_frame_2" />
   </joint>
-  <xacro:macro name="bumper" params="prefix num xyz z_dir">
-    <joint name="bumper_${prefix}_${num}_joint" type="prismatic">
-      <parent link="bumper_baseboard_${prefix}_link" />
-      <child link="bumper_${prefix}_${num}_link" />
-      <origin xyz="${xyz}" rpy="0 0 ${radians(z_dir)}" />
-      <limit lower="0.0" upper="0.0023" effort="1" velocity="1.0" />
-      <axis xyz="0 1 0" />
-      <origin xyz="0 0 0" rpy="0 0 0" />
-      <dynamics damping="0.01" />
-    </joint>
-    <transmission name="bumper_${prefix}_${num}_trans">
-      <type>transmission_interface/SimpleTransmission</type>
-      <joint name="bumper_${prefix}_${num}_joint">
-        <hardwareInterface>hardware_interface/EffortJointInterface</hardwareInterface>
-      </joint>
-      <actuator name="bumper_${prefix}_${num}_motor">
-        <hardwareInterface>hardware_interface/EffortJointInterface</hardwareInterface>
-        <mechanismReduction>1</mechanismReduction>
-      </actuator>
-    </transmission>
-    <link name="bumper_${prefix}_${num}_link">
-      <inertial>
-        <origin xyz="0 0 0" rpy="0 0 ${-radians(26)}" />
-        <mass value="0.01615" />
-        <inertia ixx="0.0000038736" iyy="0.000012239" izz="0.000014018"
-          ixy="-0.000005354147" iyz="0.000"
-          ixz="-0.000" />
-      </inertial>
-      <visual>
-        <origin xyz="0 0 0" rpy="0 0 ${-pi}" />
-        <geometry>
-          <mesh filename="package://vs_rover_options_description/meshes/bumper/mega3_bumper_link.stl" scale="0.001 0.001 0.001" />
-        </geometry>
-        <material name="silver" />
-      </visual>
-      <collision>
-        <origin xyz="0 0 0" rpy="0 0 ${-pi}" />
-        <geometry>
-          <mesh filename="package://vs_rover_options_description/meshes/bumper/mega3_bumper_link.stl" scale="0.001 0.001 0.001" />
-        </geometry>
-      </collision>
-    </link>
-    <gazebo reference="bumper_${prefix}_${num}_link">
-      <material>Gazebo/Silver</material>
-      <kp value="10000" />
-      <kd value="100" />
-    </gazebo>
+  <!-- Mega3 mounting of the reusable, passive spring-loaded 40 mm bumper. -->
+  <xacro:macro name="bumperbaseboard" params="prefix parent xyz z_dir">
+    <xacro:property name="bumper40_prefix" value="${prefix}_" />
+    <xacro:property name="bumper40_parent" value="${parent}" />
+    <xacro:property name="bumper40_xyz" value="${xyz}" />
+    <!-- The former mesh used a -pi rotation; the common model faces local +Y. -->
+    <xacro:property name="bumper40_rpy" value="0 0 ${radians(z_dir) - pi}" />
+    <xacro:include filename="$(find vs_rover_options_description)/urdf/bumper/40bumper.xacro" />
   </xacro:macro>
-  <xacro:macro name="bumperbaseboard" params="prefix parent xyz z_dir">
-    <joint name="bumper_baseboard_${prefix}_joint" type="fixed">
-      <parent link="${parent}" />
-      <child link="bumper_baseboard_${prefix}_link" />
-      <origin xyz="${xyz}" rpy="0 0 ${radians(z_dir)}" />
-    </joint>
-    <link name="bumper_baseboard_${prefix}_link">
-      <inertial>
-        <origin xyz="0 -0.018894 0.002872" rpy="0 0 0" />
-        <mass value="0.25" />
-        <inertia ixx="0.000056834" iyy="0.001431" izz="0.00148"
-          ixy="0.0" iyz="-0.000001652"
-          ixz="-0.000" />
-      </inertial>
-      <visual>
-        <origin xyz="0 0 0" rpy="0 0 ${-pi}" />
-        <geometry>
-          <mesh filename="package://vs_rover_options_description/meshes/bumper/mega3_bumper_plate.stl" scale="0.001 0.001 0.001" />
-        </geometry>
-        <material name="dark_silver" />
-      </visual>
-      <collision>
-        <origin xyz="0 0 0" rpy="0 0 ${-pi}" />
-        <geometry>
-          <mesh filename="package://vs_rover_options_description/meshes/bumper/mega3_bumper_plate.stl" scale="0.001 0.001 0.001" />
-        </geometry>
-      </collision>
-    </link>
-    <gazebo reference="bumper_baseboard_${prefix}_link">
-      <material>Gazebo/DarkGray</material>
-    </gazebo>
-    <xacro:bumper prefix="${prefix}" num="0" xyz="0.10521 -0.024711 0.0025" z_dir="26" />
-    <xacro:bumper prefix="${prefix}" num="1" xyz="0 -0.049 0.0025" z_dir="0" />
-    <xacro:bumper prefix="${prefix}" num="2" xyz="-0.10521 -0.024711 0.0025" z_dir="-26" />
-  </xacro:macro>
+  <!-- Complete product layout: including this file places all bumper assemblies. -->
+  <xacro:bumperbaseboard prefix="front" parent="base_link" xyz="0.19 0 0.02" z_dir="90" />
+  <xacro:bumperbaseboard prefix="back" parent="base_link" xyz="-0.19 0 0.02" z_dir="-90" />
 </robot>

File: urdf/bumper/bumper_x40a.xacro (robot description, xacro)
@@ -19,95 +19,26 @@
   <xacro:property name="bumper_alu_frame_z_offset" value="0.03" />
   <joint name="bumper_aluminum_frame_fixed_joint_1" type="fixed">
-    <origin xyz="${bumper_alu_frame_x_offset} 0.0 ${bumper_alu_frame_z_offset}" rpy="0 0 0" />
+    <origin xyz="0.0 ${-bumper_alu_frame_x_offset} ${bumper_alu_frame_z_offset}" rpy="0 0 ${-pi/2}" />
     <parent link="base_link" />
     <child link="bumper_aluminum_frame_1" />
   </joint>
   <joint name="bumper_aluminum_frame_fixed_joint_2" type="fixed">
-    <origin xyz="${-bumper_alu_frame_x_offset} 0.0 ${bumper_alu_frame_z_offset}" rpy="0 0 ${pi/2}" />
+    <origin xyz="0.0 ${bumper_alu_frame_x_offset} ${bumper_alu_frame_z_offset}" rpy="0 0 0" />
     <parent link="base_link" />
     <child link="bumper_aluminum_frame_2" />
   </joint>
-  <xacro:macro name="bumper" params="prefix num xyz z_dir">
-    <joint name="bumper_${prefix}_${num}_joint" type="prismatic">
-      <parent link="bumper_baseboard_${prefix}_link" />
-      <child link="bumper_${prefix}_${num}_link" />
-      <origin xyz="${xyz}" rpy="0 0 ${radians(z_dir)}" />
-      <limit lower="0.0" upper="0.0023" effort="1" velocity="1.0" />
-      <axis xyz="0 1 0" />
-      <origin xyz="0 0 0" rpy="0 0 0" />
-      <dynamics damping="0.01" />
-    </joint>
-    <transmission name="bumper_${prefix}_${num}_trans">
-      <type>transmission_interface/SimpleTransmission</type>
-      <joint name="bumper_${prefix}_${num}_joint">
-        <hardwareInterface>hardware_interface/EffortJointInterface</hardwareInterface>
-      </joint>
-      <actuator name="bumper_${prefix}_${num}_motor">
-        <hardwareInterface>hardware_interface/EffortJointInterface</hardwareInterface>
-        <mechanismReduction>1</mechanismReduction>
-      </actuator>
-    </transmission>
-    <link name="bumper_${prefix}_${num}_link">
-      <inertial>
-        <origin xyz="0 0 0" rpy="0 0 ${-radians(26)}" />
-        <mass value="0.01615" />
-        <inertia ixx="0.0000038736" iyy="0.000012239" izz="0.000014018"
-          ixy="-0.000005354147" iyz="0.000"
-          ixz="-0.000" />
-      </inertial>
-      <visual>
-        <origin xyz="0 0 0" rpy="0 0 ${-pi}" />
-        <geometry>
-          <mesh filename="package://vs_rover_options_description/meshes/bumper/x40a_bumper_link.stl" scale="0.001 0.001 0.001" />
-        </geometry>
-        <material name="silver" />
-      </visual>
-      <collision>
-        <origin xyz="0 0 0" rpy="0 0 ${-pi}" />
-        <geometry>
-          <mesh filename="package://vs_rover_options_description/meshes/bumper/x40a_bumper_link.stl" scale="0.001 0.001 0.001" />
-        </geometry>
-      </collision>
-    </link>
-    <gazebo reference="bumper_${prefix}_${num}_link">
-      <material>Gazebo/Silver</material>
-      <kp value="10000" />
-      <kd value="100" />
-    </gazebo>
+  <!-- X40A mounting of the reusable, passive spring-loaded 40 mm bumper. -->
+  <xacro:macro name="bumperbaseboard" params="prefix parent xyz z_dir">
+    <xacro:property name="bumper40_prefix" value="${prefix}_" />
+    <xacro:property name="bumper40_parent" value="${parent}" />
+    <xacro:property name="bumper40_xyz" value="${xyz}" />
+    <!-- The former mesh used a -pi rotation; the common model faces local +Y. -->
+    <xacro:property name="bumper40_rpy" value="0 0 ${radians(z_dir) - pi}" />
+    <xacro:include filename="$(find vs_rover_options_description)/urdf/bumper/40bumper.xacro" />
   </xacro:macro>
-  <xacro:macro name="bumperbaseboard" params="prefix parent xyz z_dir">
-    <joint name="bumper_baseboard_${prefix}_joint" type="fixed">
-      <parent link="${parent}" />
-      <child link="bumper_baseboard_${prefix}_link" />
-      <origin xyz="${xyz}" rpy="0 0 ${radians(z_dir)}" />
-    </joint>
-    <link name="bumper_baseboard_${prefix}_link">
-      <inertial>
-        <origin xyz="0 -0.018894 0.002872" rpy="0 0 0" />
-        <mass value="0.25" />
-        <inertia ixx="0.000056834" iyy="0.001431" izz="0.00148"
-          ixy="0.0" iyz="-0.000001652"
-          ixz="-0.000" />
-      </inertial>
-      <visual>
-        <origin xyz="0 0 0" rpy="0 0 ${-pi}" />
-        <geometry>
-          <mesh filename="package://vs_rover_options_description/meshes/bumper/x40a_bumper_plate.stl" scale="0.001 0.001 0.001" />
-        </geometry>
-        <material name="dark_silver" />
-      </visual>
-      <collision>
-        <origin xyz="0 0 0" rpy="0 0 ${-pi}" />
-        <geometry>
-          <mesh filename="package://vs_rover_options_description/meshes/bumper/x40a_bumper_plate.stl" scale="0.001 0.001 0.001" />
-        </geometry>
-      </collision>
-    </link>
-    <gazebo reference="bumper_baseboard_${prefix}_link">
-      <material>Gazebo/DarkGray</material>
-    </gazebo>
-    <xacro:bumper prefix="${prefix}" num="0" xyz="0.10521 -0.024711 0.0025" z_dir="26" />
-    <xacro:bumper prefix="${prefix}" num="1" xyz="0 -0.049 0.0025" z_dir="0" />
-    <xacro:bumper prefix="${prefix}" num="2" xyz="-0.10521 -0.024711 0.0025" z_dir="-26" />
-  </xacro:macro>
+  <!-- Complete product layout: including this file places all bumper assemblies. -->
+  <xacro:bumperbaseboard prefix="front" parent="base_link" xyz="0.20515 0 0.038" z_dir="90" />
+  <xacro:bumperbaseboard prefix="back" parent="base_link" xyz="-0.20515 0 0.038" z_dir="-90" />
+  <xacro:bumperbaseboard prefix="right" parent="base_link" xyz="0 -0.20515 0.038" z_dir="0" />
+  <xacro:bumperbaseboard prefix="left" parent="base_link" xyz="0 0.20515 0.038" z_dir="180" />
 </robot>

File: urdf/cam_stay/cam_stay_mecanum3.xacro (robot description, xacro)
@@ -4,5 +4,5 @@
   <!--　depth camera pitch angle (rad), value: 0.0 ~ 0.78 -->
   <xacro:property name="cam_pitch_angle" value="0.0" />
-  <!--　camera stay mounting position (relative to rover) x+:front, z+:up-->
+  <!--　camera stay mounting position (relative to rover) x+:front, y+:left, z+:up-->
   <xacro:property name="cam_mount_frame_x_pos" value="0.0" />
   <xacro:property name="cam_mount_frame_y_pos" value="0.0" />
@@ -13,5 +13,5 @@
 -->
   <joint name="cam_stay_frame_joint" type="fixed">
-    <origin xyz="${0.0+cam_mount_frame_y_pos} ${0.144+cam_mount_frame_x_pos} ${0.170+cam_mount_frame_z_pos}" rpy="0 0 1.5708" />
+    <origin xyz="${0.144+cam_mount_frame_x_pos} ${0.0+cam_mount_frame_y_pos} ${0.170+cam_mount_frame_z_pos}" rpy="0 0 0" />
     <parent link="base_link" />
     <child link="cam_mount_frame" />

File: urdf/cam_stay/cam_stay_x40a.xacro (robot description, xacro)
@@ -13,5 +13,5 @@
 -->
   <joint name="cam_stay_frame_joint" type="fixed">
-    <origin xyz="${0.0+cam_mount_frame_y_pos} ${0.143+cam_mount_frame_x_pos} ${0.155+cam_mount_frame_z_pos}" rpy="0 0 1.5708" />
+    <origin xyz="${0.143+cam_mount_frame_x_pos} ${-cam_mount_frame_y_pos} ${0.155+cam_mount_frame_z_pos}" rpy="0 0 ${1.5708-pi/2}" />
     <parent link="base_link" />
     <child link="cam_mount_frame" />

File: urdf/depth_cam/_d435.gazebo.xacro (robot description, xacro)
@@ -26,5 +26,6 @@
         <sensor name="${camera_name}depth" type="rgbd_camera">
         <topic>/${topics_ns}/depth</topic>
-        <gz_frame_id>${depth_optical_frame}</gz_frame_id>
+        <!-- Native RGBD XYZ uses the carrier's forward-X axes; images use optical axes. -->
+        <gz_frame_id>${reference_link}</gz_frame_id>
         <camera name="${camera_name}">
           <camera_info_topic>/${topics_ns}/depth/camera_info</camera_info_topic>

File: urdf/lrf/tg30_g120a.xacro (robot description, xacro)
@@ -1,9 +1,9 @@
 <robot name="lrf_tg30_g120a" xmlns:xacro="http://ros.org/wiki/xacro">
   <xacro:include filename="$(find vs_rover_options_description)/urdf/lrf/tg30_g120a.gazebo" />
-  <xacro:property name="tg30_lrf_front_x_offset" value="0.0" />
-  <xacro:property name="tg30_lrf_front_y_offset" value="0.29904" />
+  <xacro:property name="tg30_lrf_front_x_offset" value="0.29904" />
+  <xacro:property name="tg30_lrf_front_y_offset" value="0.0" />
   <xacro:property name="tg30_lrf_front_z_offset" value="0.1679" />
-  <xacro:property name="tg30_lrf_back_x_offset" value="0.0" />
-  <xacro:property name="tg30_lrf_back_y_offset" value="-0.29904" />
+  <xacro:property name="tg30_lrf_back_x_offset" value="-0.29904" />
+  <xacro:property name="tg30_lrf_back_y_offset" value="0.0" />
   <xacro:property name="tg30_lrf_back_z_offset" value="0.1679" />
   <xacro:property name="tg30_center_of_mass_x" value="-0.004299" />
@@ -13,5 +13,5 @@
     <parent link="base_link" />
     <child link="front_lrf_link" />
-    <origin xyz="${tg30_lrf_front_x_offset} ${tg30_lrf_front_y_offset} ${tg30_lrf_front_z_offset}" rpy="0 0 ${pi/2}" />
+    <origin xyz="${tg30_lrf_front_x_offset} ${tg30_lrf_front_y_offset} ${tg30_lrf_front_z_offset}" rpy="0 0 0" />
   </joint>
   <link name="front_lrf_link">
@@ -40,5 +40,5 @@
     <parent link="base_link" />
     <child link="back_lrf_link" />
-    <origin xyz="${tg30_lrf_back_x_offset} ${tg30_lrf_back_y_offset} ${tg30_lrf_back_z_offset}" rpy="0 0 ${-pi/2}" />
+    <origin xyz="${tg30_lrf_back_x_offset} ${tg30_lrf_back_y_offset} ${tg30_lrf_back_z_offset}" rpy="0 0 ${-pi}" />
   </joint>
   <link name="back_lrf_link">

File: urdf/lrf/tg30_g40a_lb.xacro (robot description, xacro)
@@ -1,9 +1,9 @@
 <robot name="lrf_tg30_g40a_lb" xmlns:xacro="http://ros.org/wiki/xacro">
   <xacro:include filename="$(find vs_rover_options_description)/urdf/lrf/tg30_g40a_lb.gazebo" />
-  <xacro:property name="tg30_lrf_front_x_offset" value="0.0" />
-  <xacro:property name="tg30_lrf_front_y_offset" value="0.230" />
+  <xacro:property name="tg30_lrf_front_x_offset" value="0.230" />
+  <xacro:property name="tg30_lrf_front_y_offset" value="0.0" />
   <xacro:property name="tg30_lrf_front_z_offset" value="0.0879" />
-  <xacro:property name="tg30_lrf_back_x_offset" value="0.0" />
-  <xacro:property name="tg30_lrf_back_y_offset" value="-0.230" />
+  <xacro:property name="tg30_lrf_back_x_offset" value="-0.230" />
+  <xacro:property name="tg30_lrf_back_y_offset" value="0.0" />
   <xacro:property name="tg30_lrf_back_z_offset" value="0.0879" />
   <xacro:property name="tg30_center_of_mass_x" value="-0.004299" />
@@ -13,5 +13,5 @@
     <parent link="base_link" />
     <child link="front_lrf_link" />
-    <origin xyz="${tg30_lrf_front_x_offset} ${tg30_lrf_front_y_offset} ${tg30_lrf_front_z_offset}" rpy="0 0 ${pi/2}" />
+    <origin xyz="${tg30_lrf_front_x_offset} ${tg30_lrf_front_y_offset} ${tg30_lrf_front_z_offset}" rpy="0 0 0" />
   </joint>
   <link name="front_lrf_link">
@@ -40,5 +40,5 @@
     <parent link="base_link" />
     <child link="back_lrf_link" />
-    <origin xyz="${tg30_lrf_back_x_offset} ${tg30_lrf_back_y_offset} ${tg30_lrf_back_z_offset}" rpy="0 0 ${-pi/2}" />
+    <origin xyz="${tg30_lrf_back_x_offset} ${tg30_lrf_back_y_offset} ${tg30_lrf_back_z_offset}" rpy="0 0 ${-pi}" />
   </joint>
   <link name="back_lrf_link">

File: urdf/lrf/tg30_mecanum3.xacro (robot description, xacro)
@@ -1,9 +1,9 @@
 <robot name="lrf_tg30_mecanum3" xmlns:xacro="http://ros.org/wiki/xacro">
   <xacro:include filename="$(find vs_rover_options_description)/urdf/lrf/tg30_mecanum3.gazebo" />
-  <xacro:property name="tg30_lrf_front_x_offset" value="0.0" />
-  <xacro:property name="tg30_lrf_front_y_offset" value="0.2000" />
+  <xacro:property name="tg30_lrf_front_x_offset" value="0.2000" />
+  <xacro:property name="tg30_lrf_front_y_offset" value="0.0" />
   <xacro:property name="tg30_lrf_front_z_offset" value="0.1959" />
-  <xacro:property name="tg30_lrf_back_x_offset" value="0.0" />
-  <xacro:property name="tg30_lrf_back_y_offset" value="-0.2000" />
+  <xacro:property name="tg30_lrf_back_x_offset" value="-0.2000" />
+  <xacro:property name="tg30_lrf_back_y_offset" value="0.0" />
   <xacro:property name="tg30_lrf_back_z_offset" value="0.1959" />
   <xacro:property name="tg30_center_of_mass_x" value="-0.004299" />
@@ -13,5 +13,5 @@
     <parent link="base_link" />
     <child link="front_lrf_link" />
-    <origin xyz="${tg30_lrf_front_x_offset} ${tg30_lrf_front_y_offset} ${tg30_lrf_front_z_offset}" rpy="0 0 ${pi/2}" />
+    <origin xyz="${tg30_lrf_front_x_offset} ${tg30_lrf_front_y_offset} ${tg30_lrf_front_z_offset}" rpy="0 0 0" />
   </joint>
   <link name="front_lrf_link">
@@ -40,5 +40,5 @@
     <parent link="base_link" />
     <child link="back_lrf_link" />
-    <origin xyz="${tg30_lrf_back_x_offset} ${tg30_lrf_back_y_offset} ${tg30_lrf_back_z_offset}" rpy="0 0 ${-pi/2}" />
+    <origin xyz="${tg30_lrf_back_x_offset} ${tg30_lrf_back_y_offset} ${tg30_lrf_back_z_offset}" rpy="0 0 ${-pi}" />
   </joint>
   <link name="back_lrf_link">
