Commit message: Publish verified ROS 2 Jazzy and Gazebo Harmonic package
Import the qualified package files and use the public Jazzy clone URLs.

File: urdf/lrf/tg30_x40a.xacro (robot description, xacro)
@@ -3,9 +3,9 @@
   <!-- placement of TG30 on Megarover Ver.3.0 -->
   <!-- the mesh origin is at centerline of laser, x-axis facing forward -->
-  <xacro:property name="tg30_lrf_front_x_offset" value="0" />
-  <xacro:property name="tg30_lrf_front_y_offset" value="0.234" />
+  <xacro:property name="tg30_lrf_front_x_offset" value="0.234" />
+  <xacro:property name="tg30_lrf_front_y_offset" value="0" />
   <xacro:property name="tg30_lrf_front_z_offset" value="0.2249" />
-  <xacro:property name="tg30_lrf_back_x_offset" value="0.0" />
-  <xacro:property name="tg30_lrf_back_y_offset" value="-0.234" />
+  <xacro:property name="tg30_lrf_back_x_offset" value="-0.234" />
+  <xacro:property name="tg30_lrf_back_y_offset" value="0.0" />
   <xacro:property name="tg30_lrf_back_z_offset" value="0.2249" />
   <xacro:property name="tg30_center_of_mass_x" value="-0.004299" />
@@ -16,5 +16,5 @@
     <parent link="base_link" />
     <child link="front_lrf_link" />
-    <origin xyz="${tg30_lrf_front_x_offset} ${tg30_lrf_front_y_offset} ${tg30_lrf_front_z_offset}" rpy="0 0 ${pi/2}" />
+    <origin xyz="${tg30_lrf_front_x_offset} ${tg30_lrf_front_y_offset} ${tg30_lrf_front_z_offset}" rpy="0 0 0" />
   </joint>
   <link name="front_lrf_link">
@@ -44,5 +44,5 @@
     <parent link="base_link" />
     <child link="back_lrf_link" />
-    <origin xyz="${tg30_lrf_back_x_offset} ${tg30_lrf_back_y_offset} ${tg30_lrf_back_z_offset}" rpy="0 0 ${-pi/2}" />
+    <origin xyz="${tg30_lrf_back_x_offset} ${tg30_lrf_back_y_offset} ${tg30_lrf_back_z_offset}" rpy="0 0 ${-pi}" />
   </joint>
   <link name="back_lrf_link">
